File: Kruispunt/Kruispunt schema.sch (EAGLE design)
At the start: 67 parts, among them IC1 74ACT132N, IC2 LM555N, IC3 LM555N, IC5 74AC132N, Q1 BC548, Q2 2N3906, Q5 BC548, Q6 2N3906, Q9 BC548

Commit message: Bord kruispunt + library aanpassing + logboek
Parts:
- removed IC5: 74AC132N, Kruispunt Library:74AC132N
- added C11, C8, C9: 10nF, Kruispunt Library:CERAMIC-CAP3LEADS
- added C12: 220nF, Kruispunt Library:CERAMIC-CAP3LEADS
- added D14: 1N4148DO35-7, Kruispunt Library:1N4148DO35-7
- added IC4: 74AC132N, Kruispunt Library:74AC132N
- added L2: 470µH, Detectielus library:SPOEL
- added Q10: BC548, Kruispunt Library:BC548
- added R27: 10k, Kruispunt Library:RESISTOR
- added R28: 470, Kruispunt Library:RESISTOR
- added R29: 47k, Kruispunt Library:RESISTOR
- added R30: 2,2k, Kruispunt Library:RESISTOR
- added X3: (no value), Kruispunt Library:TERMINAL-5MM-2POLE
- C7: device Detectielus library:CAPACITOR -> Kruispunt Library:CERAMIC-CAP3LEADS
- D1, D2: device Vertrangingsschema library:1N4148DO35-7 -> Kruispunt Library:1N4148DO35-7
- D10, D11, D5, D6: value 1N4148 -> 1N4148DO35-7; device Hardware lichtsturing library:1N4148DO35-7 -> Kruispunt Library:1N4148DO35-7
- D13: device Detectielus library:1N4148DO35-7 -> Kruispunt Library:1N4148DO35-7
- renumbered U$1 to ATTINY85
Connections:
- new net N$39: C8.P$1, Q10.B, R27.1, R29.2
- new net N$40: C11.P$1, C9.P$2, Q10.E, R28.1
- new net N$41: C9.P$1, L2.1, Q10.C, R30.2, X3-2.P$2
- new net N$42: C12.P$2, D14.C, IC4B.I1
- new net N$44: ATTINY85.P2, IC4B.O
- net GND: now also C11.P$2, C12.P$1, C7.P$2, C8.P$2, L2.2, R27.2, R28.2, X3-1.P$1; no longer C7.1
- net GND5: now also D14.A
- net N$31: now also C7.P$1; no longer C7.2
- net N$34: now also IC4A.I1; no longer IC5A.I1
- net N$35: now also IC4A.O; no longer IC5A.O
- net VCC: now also ATTINY85.5V, IC4A.I0, IC4B.I0; no longer IC5A.I0
- net VCC-LUS: now also R29.1, R30.1
Other:
- moved on the sheet: D10, D11, D5, D6

Commit message: Bord en schema + logboek
Parts:
- removed X1: (no value), Kruispunt Library:TERMINAL-5MM-2POLE
- added C15: 100µF, Kruispunt Library:ELCOELCO2,5MMLEAD
- added C16: 100nF, Kruispunt Library:ELCOELCO2,5MMLEAD
- added D15, D16: 1N4004, Kruispunt Library:1N4148DO35-7
- added HOLE1, HOLE2, HOLE3, HOLE4: MOUNT-HOLE-4MM, Kruispunt Library:MOUNT-HOLE-4MM
- added IC5: 786TV, Kruispunt Library:786TV
Connections:
- new net N$45: C15.+, D15.C, D16.C, IC5.VI
- net GND: now also C15.-, C16.-, IC5.GND; no longer X1-1.P$1
- net VCC: now also C16.+, D16.A, IC5.VO; no longer X5-2.P$2
- net VCC-LUS: now also D15.A, X5-2.P$2; no longer X1-2.P$2
Changed lines of the file:
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@@
 <part name="Q4" library="Kruispunt Library" deviceset="2N7000" device=""/>
 <part name="Q3" library="Kruispunt Library" deviceset="2N7000" device=""/>
-<part name="X1" library="Kruispunt Library" deviceset="TERMINAL-5MM-2POLE" device=""/>
 <part name="C2" library="Kruispunt Library" deviceset="ELCO" device="ELCO2,5MMLEAD" value="22µF"/>
 <part name="C6" library="Kruispunt Library" deviceset="ELCO" device="ELCO2,5MMLEAD" value="22µF"/>
@@
 <part name="D14" library="Kruispunt Library" deviceset="1N4148" device="DO35-7" package3d_urn="urn:adsk.eagle:package:43339/1"/>
 <part name="IC4" library="Kruispunt Library" deviceset="74*132" device="N" package3d_urn="urn:adsk.eagle:package:2008/1" technology="AC"/>
+<part name="HOLE1" library="Kruispunt Library" deviceset="MOUNT-HOLE-4MM" device=""/>
+<part name="HOLE2" library="Kruispunt Library" deviceset="MOUNT-HOLE-4MM" device=""/>
+<part name="HOLE3" library="Kruispunt Library" deviceset="MOUNT-HOLE-4MM" device=""/>
+<part name="HOLE4" library="Kruispunt Library" deviceset="MOUNT-HOLE-4MM" device=""/>
+<part name="D15" library="Kruispunt Library" deviceset="1N4148" device="DO35-7" package3d_urn="urn:adsk.eagle:package:43339/1" value="1N4004"/>
+<part name="C15" library="Kruispunt Library" deviceset="ELCO" device="ELCO2,5MMLEAD" value="100µF"/>
+<part name="C16" library="Kruispunt Library" deviceset="ELCO" device="ELCO2,5MMLEAD" value="100nF"/>
+<part name="D16" library="Kruispunt Library" deviceset="1N4148" device="DO35-7" package3d_urn="urn:adsk.eagle:package:43339/1" value="1N4004"/>
+<part name="IC5" library="Kruispunt Library" deviceset="78*" device="TV" package3d_urn="urn:adsk.eagle:package:16417/1" technology="6"/>
 </parts>
 <sheets>
@@
 <attribute name="NAME" x="344.17" y="78.74" size="1.27" layer="95" font="vector" rot="MR0"/>
 </instance>
-<instance part="X1" gate="-1" x="12.7" y="127" smashed="yes">
-<attribute name="NAME" x="11.43" y="127.889" size="1.27" layer="95" rot="R180"/>
-</instance>
-<instance part="X1" gate="-2" x="12.7" y="121.92" smashed="yes">
-<attribute name="VALUE" x="2.54" y="124.46" size="1.27" layer="96"/>
-<attribute name="NAME" x="11.43" y="122.809" size="1.27" layer="95" rot="R180"/>
-</instance>
 <instance part="C2" gate="G$1" x="297.18" y="40.64" smashed="yes">
 <attribute name="NAME" x="300.863" y="43.6626" size="1.27" layer="95" font="vector"/>
@@
 <attribute name="NAME" x="154.94" y="135.255" size="1.778" layer="95"/>
 <attribute name="VALUE" x="154.94" y="127" size="1.778" layer="96"/>
+</instance>
+<instance part="HOLE1" gate="G$1" x="15.24" y="175.26" smashed="yes">
+<attribute name="NAME" x="17.272" y="175.8442" size="1.778" layer="95"/>
+<attribute name="VALUE" x="17.272" y="172.7962" size="1.778" layer="96"/>
+</instance>
+<instance part="HOLE2" gate="G$1" x="15.24" y="167.64" smashed="yes">
+<attribute name="NAME" x="17.272" y="168.2242" size="1.778" layer="95"/>
+<attribute name="VALUE" x="17.272" y="165.1762" size="1.778" layer="96"/>
+</instance>
+<instance part="HOLE3" gate="G$1" x="15.24" y="160.02" smashed="yes">
+<attribute name="NAME" x="17.272" y="160.6042" size="1.778" layer="95"/>
+<attribute name="VALUE" x="17.272" y="157.5562" size="1.778" layer="96"/>
+</instance>
+<instance part="HOLE4" gate="G$1" x="15.24" y="152.4" smashed="yes">
+<attribute name="NAME" x="17.272" y="152.9842" size="1.778" layer="95"/>
+<attribute name="VALUE" x="17.272" y="149.9362" size="1.778" layer="96"/>
+</instance>
+<instance part="D15" gate="G$1" x="223.52" y="177.8" smashed="yes">
+<attribute name="NAME" x="226.06" y="178.2826" size="1.778" layer="95"/>
+<attribute name="VALUE" x="226.06" y="175.4886" size="1.778" layer="96"/>
+</instance>
+<instance part="C15" gate="G$1" x="233.68" y="167.64" smashed="yes">
+<attribute name="NAME" x="234.823" y="170.6626" size="1.27" layer="95" font="vector"/>
+<attribute name="VALUE" x="234.823" y="165.5826" size="1.27" layer="96" font="vector"/>
+</instance>
+<instance part="C16" gate="G$1" x="261.62" y="167.64" smashed="yes">
+<attribute name="NAME" x="262.763" y="170.6626" size="1.27" layer="95" font="vector"/>
+<attribute name="VALUE" x="262.763" y="165.5826" size="1.27" layer="96" font="vector"/>
+</instance>
+<instance part="D16" gate="G$1" x="248.92" y="193.04" smashed="yes" rot="R180">
+<attribute name="NAME" x="246.38" y="192.5574" size="1.778" layer="95" rot="R180"/>
+<attribute name="VALUE" x="246.38" y="195.3514" size="1.778" layer="96" rot="R180"/>
+</instance>
+<instance part="IC5" gate="A1" x="248.92" y="177.8" smashed="yes">
+<attribute name="NAME" x="241.3" y="183.515" size="1.778" layer="95"/>
+<attribute name="VALUE" x="241.3" y="180.975" size="1.778" layer="96"/>
 </instance>
 </instances>
@@
 </segment>
 <segment>
-<pinref part="X1" gate="-1" pin="P$1"/>
-<wire x1="17.78" y1="127" x2="22.86" y2="127" width="0.1524" layer="91"/>
-<label x="20.32" y="127" size="1.778" layer="95"/>
-</segment>
-<segment>
 <wire x1="78.74" y1="109.22" x2="78.74" y2="106.68" width="0.1524" layer="91"/>
 <wire x1="78.74" y1="106.68" x2="63.5" y2="106.68" width="0.1524" layer="91"/>
@@
 <junction x="111.76" y="111.76"/>
 </segment>
+<segment>
+<pinref part="C15" gate="G$1" pin="-"/>
+<wire x1="233.68" y1="165.1" x2="233.68" y2="162.56" width="0.1524" layer="91"/>
+<wire x1="233.68" y1="162.56" x2="193.04" y2="162.56" width="0.1524" layer="91"/>
+<wire x1="248.92" y1="170.18" x2="248.92" y2="162.56" width="0.1524" layer="91"/>
+<wire x1="248.92" y1="162.56" x2="233.68" y2="162.56" width="0.1524" layer="91"/>
+<junction x="233.68" y="162.56"/>
+<pinref part="C16" gate="G$1" pin="-"/>
+<wire x1="261.62" y1="165.1" x2="261.62" y2="162.56" width="0.1524" layer="91"/>
+<wire x1="261.62" y1="162.56" x2="248.92" y2="162.56" width="0.1524" layer="91"/>
+<junction x="248.92" y="162.56"/>
+<wire x1="261.62" y1="162.56" x2="289.56" y2="162.56" width="0.1524" layer="91"/>
+<junction x="261.62" y="162.56"/>
+<label x="198.12" y="162.56" size="1.778" layer="95"/>
+<label x="274.32" y="162.56" size="1.778" layer="95"/>
+<pinref part="IC5" gate="A1" pin="GND"/>
+</segment>
 </net>
 <net name="N$7" class="0">
@@
 </net>
 <net name="VCC" class="0">
-<segment>
-<pinref part="X5" gate="-2" pin="P$2"/>
-<wire x1="17.78" y1="105.41" x2="21.59" y2="105.41" width="0.1524" layer="91"/>
-<label x="19.05" y="105.41" size="1.778" layer="95"/>
-</segment>
 <segment>
 <wire x1="182.88" y1="99.06" x2="182.88" y2="111.76" width="0.1524" layer="91"/>
@@
 <wire x1="132.08" y1="134.62" x2="144.78" y2="134.62" width="0.1524" layer="91"/>
 <pinref part="IC4" gate="B" pin="I0"/>
+</segment>
+<segment>
+<pinref part="C16" gate="G$1" pin="+"/>
+<wire x1="261.62" y1="172.72" x2="261.62" y2="177.8" width="0.1524" layer="91"/>
+<wire x1="261.62" y1="177.8" x2="289.56" y2="177.8" width="0.1524" layer="91"/>
+<label x="274.32" y="177.8" size="1.778" layer="95"/>
+<pinref part="IC5" gate="A1" pin="VO"/>
+<wire x1="259.08" y1="177.8" x2="261.62" y2="177.8" width="0.1524" layer="91"/>
+<junction x="261.62" y="177.8"/>
+<pinref part="D16" gate="G$1" pin="A"/>
+<wire x1="261.62" y1="193.04" x2="251.46" y2="193.04" width="0.1524" layer="91"/>
+<wire x1="261.62" y1="193.04" x2="261.62" y2="177.8" width="0.1524" layer="91"/>
 </segment>
 </net>
@@
 </segment>
 <segment>
-<pinref part="X1" gate="-2" pin="P$2"/>
-<wire x1="17.78" y1="121.92" x2="22.86" y2="121.92" width="0.1524" layer="91"/>
-<label x="20.32" y="121.92" size="1.778" layer="95"/>
-</segment>
-<segment>
 <wire x1="63.5" y1="154.94" x2="63.5" y2="157.48" width="0.1524" layer="91"/>
 <wire x1="63.5" y1="157.48" x2="71.12" y2="157.48" width="0.1524" layer="91"/>
@@
 <pinref part="R29" gate="G$1" pin="1"/>
 <pinref part="R30" gate="G$1" pin="1"/>
+</segment>
+<segment>
+<wire x1="193.04" y1="177.8" x2="220.98" y2="177.8" width="0.1524" layer="91"/>
+<label x="198.12" y="177.8" size="1.778" layer="95"/>
+<pinref part="D15" gate="G$1" pin="A"/>
+</segment>
+<segment>
+<pinref part="X5" gate="-2" pin="P$2"/>
+<wire x1="17.78" y1="105.41" x2="21.59" y2="105.41" width="0.1524" layer="91"/>
+<label x="19.05" y="105.41" size="1.778" layer="95"/>
 </segment>
 </net>
@@
 </segment>
 </net>
+<net name="N$45" class="0">
+<segment>
+<pinref part="D16" gate="G$1" pin="C"/>
+<wire x1="246.38" y1="193.04" x2="233.68" y2="193.04" width="0.1524" layer="91"/>
+<pinref part="D15" gate="G$1" pin="C"/>
+<wire x1="226.06" y1="177.8" x2="233.68" y2="177.8" width="0.1524" layer="91"/>
+<pinref part="C15" gate="G$1" pin="+"/>
+<wire x1="233.68" y1="172.72" x2="233.68" y2="177.8" width="0.1524" layer="91"/>
+<pinref part="IC5" gate="A1" pin="VI"/>
+<wire x1="238.76" y1="177.8" x2="233.68" y2="177.8" width="0.1524" layer="91"/>
+<junction x="233.68" y="177.8"/>
+<wire x1="233.68" y1="193.04" x2="233.68" y2="177.8" width="0.1524" layer="91"/>
+</segment>
+</net>
