File: Kruispunt/Kruispunt schema.sch (EAGLE design)
At the start: 115 parts, among them IC1 74ACT132N, IC2 LM555N, IC3 LM555N, IC4 74AC132N, Q1 BC548, Q10 BC548, Q2 2N3906, Q5 BC548, Q6 2N3906, Q9 BC548

Commit message: Schema en ppt
Parts:
- X1: value (none) -> Rood2
- X10: value (none) -> Voetgagnersknop1
- X11: value (none) -> Voetgangersknop2
- X12: value (none) -> Groen1
- X13: value (none) -> Geel1
- X14: value (none) -> Groen2
- X4: value (none) -> Rood1
- X6: value (none) -> Geel2
Changed lines of the file:
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@@
 <?xml version="1.0" encoding="utf-8"?>
 <!DOCTYPE eagle SYSTEM "eagle.dtd">
-<eagle version="9.2.2">
+<eagle version="9.1.2">
 <drawing>
 <settings>
@@
 <part name="SUPPLY14" library="Vertrangingsschema library" deviceset="GND5" device="" value="GND"/>
 <part name="SUPPLY15" library="Vertrangingsschema library" deviceset="GND5" device="" value="GND"/>
-<part name="X10" library="Kruispunt Library" deviceset="TERMINAL-5MM-2POLE" device=""/>
-<part name="X11" library="Kruispunt Library" deviceset="TERMINAL-5MM-2POLE" device=""/>
-<part name="X4" library="Kruispunt Library" deviceset="TERMINAL-5MM-2POLE" device=""/>
-<part name="X12" library="Kruispunt Library" deviceset="TERMINAL-5MM-2POLE" device=""/>
-<part name="X13" library="Kruispunt Library" deviceset="TERMINAL-5MM-2POLE" device=""/>
-<part name="X1" library="Kruispunt Library" deviceset="TERMINAL-5MM-2POLE" device=""/>
-<part name="X6" library="Kruispunt Library" deviceset="TERMINAL-5MM-2POLE" device=""/>
-<part name="X14" library="Kruispunt Library" deviceset="TERMINAL-5MM-2POLE" device=""/>
+<part name="X10" library="Kruispunt Library" deviceset="TERMINAL-5MM-2POLE" device="" value="Voetgagnersknop1"/>
+<part name="X11" library="Kruispunt Library" deviceset="TERMINAL-5MM-2POLE" device="" value="Voetgangersknop2"/>
+<part name="X4" library="Kruispunt Library" deviceset="TERMINAL-5MM-2POLE" device="" value="Rood1"/>
+<part name="X12" library="Kruispunt Library" deviceset="TERMINAL-5MM-2POLE" device="" value="Groen1"/>
+<part name="X13" library="Kruispunt Library" deviceset="TERMINAL-5MM-2POLE" device="" value="Geel1"/>
+<part name="X1" library="Kruispunt Library" deviceset="TERMINAL-5MM-2POLE" device="" value="Rood2"/>
+<part name="X6" library="Kruispunt Library" deviceset="TERMINAL-5MM-2POLE" device="" value="Geel2"/>
+<part name="X14" library="Kruispunt Library" deviceset="TERMINAL-5MM-2POLE" device="" value="Groen2"/>
 </parts>
 <sheets>
@@
 </instance>
 <instance part="X4" gate="-2" x="375.92" y="104.14" smashed="yes" rot="R180">
-<attribute name="VALUE" x="386.08" y="101.6" size="1.27" layer="96" rot="R180"/>
+<attribute name="VALUE" x="382.27" y="99.822" size="1.27" layer="96" rot="R180"/>
 <attribute name="NAME" x="377.19" y="103.251" size="1.27" layer="95"/>
 </instance>
@@
 </instance>
 <instance part="X12" gate="-2" x="355.6" y="35.56" smashed="yes">
-<attribute name="VALUE" x="345.44" y="38.1" size="1.27" layer="96"/>
+<attribute name="VALUE" x="349.758" y="39.878" size="1.27" layer="96"/>
 <attribute name="NAME" x="354.33" y="36.449" size="1.27" layer="95" rot="R180"/>
 </instance>
@@
 </instance>
 <instance part="X13" gate="-2" x="401.32" y="60.96" smashed="yes" rot="R270">
-<attribute name="VALUE" x="403.86" y="71.12" size="1.27" layer="96" rot="R270"/>
+<attribute name="VALUE" x="405.638" y="66.548" size="1.27" layer="96" rot="R270"/>
 <attribute name="NAME" x="402.209" y="62.23" size="1.27" layer="95" rot="R90"/>
 </instance>

Commit message: Schema, gerber, logboek
Parts:
- X11: value Voetgangersknop2 -> Voetgangersknop 2 en 1
Connections:
- removed net DIG-IN: C1.P$2, C5.P$2, D1.C, D11.C, D12.A, D2.C, D6.C, D7.A, IC1B.O, IC1C.O, PAD1.MOUNT, PAD2.MOUNT, Q3.G, Q7.G, R11.2, R15.1, R17.2, R23.S, R24.S, R3.1, R8.1, R9.1, X13-1.P$1, X6-1.P$1
- new net DIG-IN1: C1.P$2, D1.C, D6.C, D7.A, IC1C.O, PAD1.MOUNT, Q3.G, R24.S, R3.1, R8.1, R9.1, X13-1.P$1
- new net DIG-IN2: C5.P$2, D11.C, D12.A, D2.C, IC1B.O, PAD2.MOUNT, Q7.G, R11.2, R15.1, R17.2, R23.S, X6-1.P$1
