File: Kruispunt/Kruispunt schema v2.brd (EAGLE design)
At the start: 100 x 100.1 mm, 115 parts, among them IC1 74ACT132N, IC2 LM555N, IC3 LM555N, IC4 74AC132N, Q1 BC548, Q10 BC548, Q2 2N3906, Q5 BC548, Q6 2N3906, Q9 BC548, X1 Rood2, X10 Voetgagnersknop1, X11 Voetgangersknop 2 en 1, X12 Groen1, X13 Geel1, X14 Groen2, X4 Rood1, X6 Geel2

Commit message: kruispunt
Parts:
- added PAD18, PAD19: Meetpin, Kruispunt Library:PAD
Connections:
- removed net N$16 (its old number): D5.C, D6.C, Q4.2, R9.2
- removed net N$3 (its old number): C3.+, D1.A, IC1.5, R1.1
- new net N$1: C4.+, D2.A, IC1.5, R2.1
- new net N$41: D5.A, D6.A, Q4.2, R9.2
- net DIG-IN1: now also D2.C, D6.C, R23.2; no longer D1.C, D6.A, R24.2, R9.1
- net DIG-IN2: now also D1.C, D11.C, R24.2; no longer D11.A, D2.C, R17.2, R23.2
- net N$15: now also D5.C; no longer D5.A
- net N$27: now also D10.C; no longer D10.A
- net N$28: now also D10.A, D11.A; no longer D10.C, D11.C
- net N$34: now also PAD18.P$1
- net N$42: now also PAD19.P$1
- net N$7: now also C3.+, D1.A, R1.1; no longer C4.+, D2.A, R2.1
- net VCC: now also R17.2, R9.1

Commit message: kruispunt
Parts:
- removed L1, L2: 470µH, Detectielus library:IR-4
- removed PAD1, PAD10, PAD11, PAD12, PAD13, PAD15, PAD17, PAD18, PAD19, PAD2, PAD5, PAD9: Meetpin, Kruispunt Library:PAD
- added 1, 10, 11, 15, 17, 2, 5, 9: Meetpin, Kruispunt Library:PAD
- added 12, 13, 18, 19: (no value), Kruispunt Library:PAD
- added D17, D18: 1N821, Kruispunt Library:DO35Z10
- added JP1, JP2: (no value), Kruispunt Library:1X02
- added X7, X8, X9: (no value), Kruispunt Library:W237-132
- C1, C11, C13, C14, C17, C18, C19, C5, C7, C8, C9: device Kruispunt Library:CERAMIC-CAP-C025_050-035X075 -> test(3):CERAMIC-CAP-C050-025X075
- moved IC4 14.4 mm to (84.8, 52.8)
- moved C10 12.0 mm to (87.9, 71.7)
- moved D14 8.25 mm to (76.8, 40.2)
- moved D13 7.28 mm to (72.8, 40.0)
- moved C11 6.08 mm to (81.9, 72.4)
- moved Q2 4.12 mm to (41.1, 32.7)
- moved Q9 3.65 mm to (56.5, 50.1), turned to 90 degrees
- moved Q10 3.64 mm to (63.5, 50.1), turned to 90 degrees
- moved D16 2.00 mm to (84.3, 22.1)
- moved C1 1.00 mm to (40.6, 40.6)
- moved C19 1.00 mm to (4.92, 3.81)
- moved D15 1.00 mm to (84.3, 27.5)
- renumbered PAD14 to 14, PAD16 to 16, PAD3 to 3, PAD4 to 4, PAD6 to 6, PAD7 to 7, PAD8 to 8
Connections:
- new net N$47: 2.P$1, D1.C, IC1.6, JP2.1, R24.2
- new net N$48: ATTINY85.P2, X8.2
- new net N$50: ATTINY85.P0, X8.1
- new net N$6: 1.P$1, D2.C, IC1.8, JP1.1, R23.2
- net DIG-IN1: now also JP1.2; no longer C1.P$3, D2.C, IC1.8, PAD1.P$1, R23.2
- net DIG-IN2: now also JP2.2; no longer C5.P$3, D1.C, IC1.6, PAD2.P$1, R24.2
- net GND: now also 11.P$1, D17.A, D18.A, X12.1, X14.1, X9.1; no longer PAD11.P$1, X12.2, X14.2
- net LUS-OUT1: no longer L2.1
- net N$10: now also 17.P$1; no longer PAD17.P$1
- net N$11: now also X12.2; no longer X12.1
- net N$13: now also 12.P$1; no longer PAD12.P$1
- net N$17: now also 13.P$1; no longer PAD13.P$1
- net N$20: now also 5.P$1; no longer PAD5.P$1
- net N$23: now also X14.2; no longer X14.1
- net N$29: now also 15.P$1; no longer PAD15.P$1
- net N$32: no longer C13.P$3
- net N$33: no longer L1.1
- net N$34: now also 18.P$1, D18.C; no longer PAD18.P$1
- net N$35: now also X7.2; no longer ATTINY85.P0
- net N$38: no longer C19.P$3
- net N$40: no longer C9.P$3
- net N$42: now also 19.P$1, D17.C; no longer PAD19.P$1
- net N$43: no longer C18.P$3
- net N$44: now also X7.1; no longer ATTINY85.P2
- net N48: no longer C11.P$3, C8.P$3, L2.2
- net N49: no longer C14.P$3, C7.P$3, L1.2
- net VCC: now also 10.P$1, X9.2; no longer C17.P$3, PAD10.P$1
- net VCC-LUS: now also 9.P$1; no longer PAD9.P$1
Routing:
- net VCC: track 0.00 -> 463.9 mm, vias 0 -> 3
- net N$26: track 0.00 -> 177.6 mm
- net N$18: track 0.00 -> 155.1 mm
- net N$47: track 0.00 -> 142.3 mm, vias 0 -> 2
- net N$46: track 0.00 -> 128.9 mm, vias 0 -> 4
- net N$14: track 0.00 -> 128.1 mm, vias 0 -> 2
- net N$6: track 0.00 -> 127.9 mm, vias 0 -> 1
- net N$44: track 0.00 -> 127.5 mm, vias 0 -> 2
- net N$48: track 0.00 -> 116.6 mm, vias 0 -> 2
- net DIG-IN1: track 0.00 -> 111.5 mm, vias 0 -> 2
- net N$11: track 0.00 -> 108.4 mm, vias 0 -> 3
- net N$35: track 0.00 -> 96.9 mm, vias 0 -> 1
- net VCC-LUS: track 0.00 -> 94.0 mm, vias 0 -> 1
- net N$50: track 0.00 -> 93.4 mm, vias 0 -> 2
- net N$20: track 0.00 -> 87.7 mm, vias 0 -> 1
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Other:
- board text added: "Kruispunt V2 Robbe Dierickx 21/02/2019"
- board text added: "VCC"
- board text removed: "Kruispunt V1 Robbe Dierickx 11/01/19"

Commit message: v3
Connections:
- net DIG-IN1: now also R3.2; no longer R3.1
- net DIG-IN2: now also R11.1; no longer R11.2
- net GND: now also R11.2, R3.1
- net VCC: no longer R11.1, R3.2
Routing:
- net VCC: track 463.9 -> 0.00 mm, vias 3 -> 0
- net N$26: track 177.6 -> 0.00 mm
- net N$18: track 155.1 -> 0.00 mm
- net N$47: track 142.3 -> 0.00 mm, vias 2 -> 0
- net N$46: track 128.9 -> 0.00 mm, vias 4 -> 0
- net N$14: track 128.1 -> 0.00 mm, vias 2 -> 0
- net N$6: track 127.9 -> 0.00 mm, vias 1 -> 0
- net N$44: track 127.5 -> 0.00 mm, vias 2 -> 0
- net N$48: track 116.6 -> 0.00 mm, vias 2 -> 0
- net DIG-IN1: track 111.5 -> 0.00 mm, vias 2 -> 0
- net N$11: track 108.4 -> 0.00 mm, vias 3 -> 0
- net N$35: track 96.9 -> 0.00 mm, vias 1 -> 0
- net VCC-LUS: track 94.0 -> 0.00 mm, vias 1 -> 0
- net N$50: track 93.4 -> 0.00 mm, vias 2 -> 0
- net N$20: track 87.7 -> 0.00 mm, vias 1 -> 0
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