File: Kruispunt/Kruispunt schema v2.sch (EAGLE design)
At the start: 107 parts, among them IC1 74ACT132N, IC2 LM555N, IC3 LM555N, IC4 74AC132N, Q1 BC548, Q10 BC548, Q2 2N3906, Q5 BC548, Q6 2N3906, Q9 BC548

Commit message: schema v2
Parts:
- added X1: Rood2, Kruispunt Library:TERMINAL-5MM-2POLE
- added X10: Voetgagnersknop1, Kruispunt Library:TERMINAL-5MM-2POLE
- added X11: Voetgangersknop 2 en 1, Kruispunt Library:TERMINAL-5MM-2POLE
- added X12: Groen1, Kruispunt Library:TERMINAL-5MM-2POLE
- added X13: Geel1, Kruispunt Library:TERMINAL-5MM-2POLE
- added X14: Groen2, Kruispunt Library:TERMINAL-5MM-2POLE
- added X4: Rood1, Kruispunt Library:TERMINAL-5MM-2POLE
- added X6: Geel2, Kruispunt Library:TERMINAL-5MM-2POLE
Connections:
- removed net DIG-IN: C1.P$2, C5.P$2, D1.C, D11.C, D12.A, D2.C, D6.C, D7.A, IC1B.O, IC1C.O, PAD1.MOUNT, PAD2.MOUNT, Q3.G, Q7.G, R11.2, R15.1, R17.2, R23.S, R24.S, R3.1, R8.1, R9.1
- removed net GND5: D13.A, D14.A
- removed net N$41: C9.P$1, L2.1, Q10.C, R30.2, X3-2.P$2
- new net DIG-IN1: C1.P$2, D1.C, D6.A, IC1C.O, PAD1.MOUNT, Q3.G, R24.S, R3.1, R8.1, R9.1
- new net DIG-IN2: C5.P$2, D11.A, D2.C, IC1B.O, PAD2.MOUNT, Q7.G, R11.2, R15.1, R17.2, R23.S
- new net LUS-OUT1: C12.P$1, C9.P$1, L2.1, Q10.C, R30.2, X3-2.P$2
- new net N$46: ATTINY85.P4, X11-2.P$2
- new net N$49: D9.C, R16.1, X1-1.P$1
- new net N48: C11.P$2, C8.P$2, L2.2, X3-1.P$1
- new net N49: C14.P$2, C7.P$2, L1.2, X2-1.P$1
- net GND: now also D13.A, D14.A, X10-1.P$1, X11-1.P$1, X12-2.P$2, X14-2.P$2; no longer C10.P$1, C11.P$2, C12.P$1, C14.P$2, C7.P$2, C8.P$2, L1.2, L2.2, X2-1.P$1, X3-1.P$1
- net N$11: now also X12-1.P$1
- net N$14: now also X4-1.P$1
- net N$15: now also D5.A; no longer D5.C
- net N$16: now also D5.C, D6.C; no longer D5.A, D6.A
- net N$18: now also X13-2.P$2
- net N$23: now also X14-1.P$1
- net N$26: now also ATTINY85.P3, X10-2.P$2; no longer D9.C, R16.1
- net N$27: now also D10.A; no longer D10.C
- net N$28: now also D10.C, D11.C; no longer D10.A, D11.A
- net N$30: now also X6-2.P$2
- net N$33: now also C10.P$1
- net VCC: now also D12.A, D7.A, X1-2.P$2, X13-1.P$1, X4-2.P$2, X6-1.P$1
Other:
- moved on the sheet: C10, C12, D13, D14

Commit message: kruispunt
Parts:
- added PAD18, PAD19: Meetpin, Kruispunt Library:WIREPAD
Connections:
- removed net N$16 (its old number): D5.C, D6.C, Q4.G, R9.2
- removed net N$3 (its old number): C3.+, D1.A, IC1B.I1, R1.1
- new net N$1: C4.+, D2.A, IC1B.I1, R2.1
- new net N$41: D5.A, D6.A, Q4.G, R9.2
- net DIG-IN1: now also D2.C, D6.C, R23.S; no longer D1.C, D6.A, R24.S, R9.1
- net DIG-IN2: now also D1.C, D11.C, R24.S; no longer D11.A, D2.C, R17.2, R23.S
- net N$15: now also D5.C; no longer D5.A
- net N$27: now also D10.C; no longer D10.A
- net N$28: now also D10.A, D11.A; no longer D10.C, D11.C
- net N$34: now also PAD18.MOUNT
- net N$42: now also PAD19.MOUNT
- net N$7: now also C3.+, D1.A, R1.1; no longer C4.+, D2.A, R2.1
- net VCC: now also R17.2, R9.1
Other:
- moved on the sheet: C3, C4, D1, D10, D11, D2, D5, D6, IC1B, R1, R2, R23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

Commit message: kruispunt
Parts:
- removed L1, L2: 470µH, Detectielus library:SPOEL
- added D17, D18: 1N821, Kruispunt Library:1N821
- added JP1, JP2: (no value), Kruispunt Library:PINHD-1X2
- added X7, X8, X9: (no value), Kruispunt Library:TERMINAL-5MM-2POLE
- 12, 13, 18, 19: value Meetpin -> WIREPAD
- C1, C11, C13, C14, C17, C18, C19, C5, C7, C8, C9: device Kruispunt Library:CERAMIC-CAP3LEADS -> test(3):CERAMIC-CAP2LEADS
- renumbered PAD1 to 1, PAD10 to 10, PAD11 to 11, PAD12 to 12, PAD13 to 13, PAD14 to 14, PAD15 to 15, PAD16 to 16, PAD17 to 17, PAD18 to 18, PAD19 to 19, PAD2 to 2, PAD3 to 3, PAD4 to 4, PAD5 to 5, PAD6 to 6, PAD7 to 7, PAD8 to 8, PAD9 to 9
Connections:
- new net N$47: 2.MOUNT, D1.C, IC1B.O, JP2.1, R24.S
- new net N$48: ATTINY85.P2, X8-2.P$2
- new net N$50: ATTINY85.P0, X8-1.P$1
- new net N$6: 1.MOUNT, D2.C, IC1C.O, JP1.1, R23.S
- net DIG-IN1: now also JP1.2; no longer 1.MOUNT, D2.C, IC1C.O, R23.S
- net DIG-IN2: now also JP2.2; no longer 2.MOUNT, D1.C, IC1B.O, R24.S
- net GND: now also D17.A, D18.A, X12-1.P$1, X14-1.P$1, X9-1.P$1; no longer X12-2.P$2, X14-2.P$2
- net LUS-OUT1: no longer L2.1
- net N$11: now also X12-2.P$2; no longer X12-1.P$1
- net N$23: now also X14-2.P$2; no longer X14-1.P$1
- net N$33: no longer L1.1
- net N$34: now also D18.C
- net N$35: now also X7-2.P$2; no longer ATTINY85.P0
- net N$42: now also D17.C
- net N$44: now also X7-1.P$1; no longer ATTINY85.P2
- net N48: no longer L2.2
- net N49: no longer L1.2
- net VCC: now also X9-2.P$2
Other:
- moved on the sheet: X12-1, X12-2, X14-1, X14-2

Commit message: v3
Connections:
- net DIG-IN1: now also R3.2; no longer R3.1
- net DIG-IN2: now also R11.1; no longer R11.2
- net GND: now also R11.2, R3.1
- net VCC: no longer R11.1, R3.2
Other:
- moved on the sheet: R11, R3
Changed lines of the file:
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@@
 <attribute name="VALUE" x="267.462" y="92.71" size="1.778" layer="96" rot="R90"/>
 </instance>
-<instance part="R3" gate="G$1" x="215.9" y="93.98" smashed="yes" rot="R90">
-<attribute name="NAME" x="214.4014" y="90.17" size="1.778" layer="95" rot="R90"/>
-<attribute name="VALUE" x="219.202" y="90.17" size="1.778" layer="96" rot="R90"/>
+<instance part="R3" gate="G$1" x="215.9" y="50.8" smashed="yes" rot="R90">
+<attribute name="NAME" x="214.4014" y="46.99" size="1.778" layer="95" rot="R90"/>
+<attribute name="VALUE" x="219.202" y="46.99" size="1.778" layer="96" rot="R90"/>
 </instance>
 <instance part="R6" gate="G$1" x="360.68" y="91.44" smashed="yes" rot="R90">
@@
 <attribute name="VALUE" x="403.098" y="100.33" size="1.778" layer="96" rot="R270"/>
 </instance>
-<instance part="R11" gate="G$1" x="185.42" y="-25.4" smashed="yes" rot="R270">
-<attribute name="NAME" x="186.9186" y="-21.59" size="1.778" layer="95" rot="R270"/>
-<attribute name="VALUE" x="182.118" y="-21.59" size="1.778" layer="96" rot="R270"/>
+<instance part="R11" gate="G$1" x="185.42" y="-60.96" smashed="yes" rot="R270">
+<attribute name="NAME" x="186.9186" y="-57.15" size="1.778" layer="95" rot="R270"/>
+<attribute name="VALUE" x="182.118" y="-57.15" size="1.778" layer="96" rot="R270"/>
 </instance>
 <instance part="R12" gate="G$1" x="233.68" y="-22.86" smashed="yes" rot="R270">
@@
 <pinref part="X12" gate="-1" pin="P$1"/>
 <wire x1="360.68" y1="35.56" x2="363.22" y2="35.56" width="0.1524" layer="91"/>
+<pinref part="R3" gate="G$1" pin="1"/>
+<wire x1="215.9" y1="45.72" x2="215.9" y2="30.48" width="0.1524" layer="91"/>
+<wire x1="215.9" y1="30.48" x2="264.16" y2="30.48" width="0.1524" layer="91"/>
+<junction x="264.16" y="30.48"/>
 </segment>
 <segment>
@@
 <pinref part="X14" gate="-1" pin="P$1"/>
 <wire x1="332.74" y1="-83.82" x2="333.756" y2="-83.82" width="0.1524" layer="91"/>
+<pinref part="R11" gate="G$1" pin="2"/>
+<wire x1="185.42" y1="-66.04" x2="185.42" y2="-88.9" width="0.1524" layer="91"/>
+<wire x1="185.42" y1="-88.9" x2="233.68" y2="-88.9" width="0.1524" layer="91"/>
+<junction x="233.68" y="-88.9"/>
 </segment>
 <segment>
@@
 <net name="VCC" class="1">
 <segment>
-<wire x1="215.9" y1="99.06" x2="215.9" y2="111.76" width="0.1524" layer="91"/>
-<wire x1="215.9" y1="111.76" x2="264.16" y2="111.76" width="0.1524" layer="91"/>
 <wire x1="264.16" y1="111.76" x2="264.16" y2="101.6" width="0.1524" layer="91"/>
 <pinref part="SUPPLY3" gate="G$1" pin="VCC"/>
 <wire x1="295.91" y1="129.54" x2="295.91" y2="111.76" width="0.1524" layer="91"/>
 <wire x1="295.91" y1="111.76" x2="264.16" y2="111.76" width="0.1524" layer="91"/>
-<junction x="264.16" y="111.76"/>
 <pinref part="IC2" gate="A" pin="V+"/>
 <wire x1="320.04" y1="57.15" x2="325.12" y2="57.15" width="0.1524" layer="91"/>
@@
 <wire x1="360.68" y1="106.68" x2="360.68" y2="109.22" width="0.1524" layer="91"/>
 <label x="309.88" y="111.76" size="1.778" layer="95"/>
-<pinref part="R3" gate="G$1" pin="2"/>
 <pinref part="R4" gate="G$1" pin="2"/>
 <wire x1="360.68" y1="109.22" x2="360.68" y2="111.76" width="0.1524" layer="91"/>
@@
 </segment>
 <segment>
-<wire x1="185.42" y1="-20.32" x2="185.42" y2="-7.62" width="0.1524" layer="91"/>
-<wire x1="185.42" y1="-7.62" x2="233.68" y2="-7.62" width="0.1524" layer="91"/>
 <wire x1="233.68" y1="-7.62" x2="233.68" y2="-17.78" width="0.1524" layer="91"/>
 <pinref part="SUPPLY4" gate="G$1" pin="VCC"/>
 <wire x1="265.43" y1="10.16" x2="265.43" y2="-7.62" width="0.1524" layer="91"/>
 <wire x1="265.43" y1="-7.62" x2="233.68" y2="-7.62" width="0.1524" layer="91"/>
-<junction x="233.68" y="-7.62"/>
 <pinref part="IC3" gate="A" pin="V+"/>
 <wire x1="289.56" y1="-62.23" x2="294.64" y2="-62.23" width="0.1524" layer="91"/>
@@
 <wire x1="330.2" y1="-12.7" x2="330.2" y2="-10.668" width="0.1524" layer="91"/>
 <label x="279.4" y="-7.62" size="1.778" layer="95"/>
-<pinref part="R11" gate="G$1" pin="1"/>
 <pinref part="R12" gate="G$1" pin="1"/>
 <wire x1="330.2" y1="-10.668" x2="330.2" y2="-7.62" width="0.1524" layer="91"/>
@@
 <segment>
 <wire x1="177.8" y1="-45.72" x2="185.42" y2="-45.72" width="0.1524" layer="91"/>
-<wire x1="185.42" y1="-30.48" x2="185.42" y2="-33.02" width="0.1524" layer="91"/>
 <junction x="185.42" y="-45.72"/>
 <wire x1="185.42" y1="-33.02" x2="185.42" y2="-45.72" width="0.1524" layer="91"/>
-<wire x1="185.42" y1="-33.02" x2="193.04" y2="-33.02" width="0.1524" layer="91"/>
-<junction x="185.42" y="-33.02"/>
-<wire x1="193.04" y1="-33.02" x2="193.04" y2="-2.54" width="0.1524" layer="91"/>
-<wire x1="193.04" y1="-2.54" x2="358.14" y2="-2.54" width="0.1524" layer="91"/>
+<wire x1="185.42" y1="-33.02" x2="185.42" y2="-2.54" width="0.1524" layer="91"/>
+<wire x1="185.42" y1="-2.54" x2="358.14" y2="-2.54" width="0.1524" layer="91"/>
 <wire x1="358.14" y1="-2.54" x2="358.14" y2="-43.18" width="0.1524" layer="91"/>
 <wire x1="358.14" y1="-43.18" x2="358.14" y2="-48.26" width="0.1524" layer="91"/>
@@
 <pinref part="Q7" gate="G$1" pin="G"/>
 <wire x1="342.9" y1="-43.18" x2="358.14" y2="-43.18" width="0.1524" layer="91"/>
-<pinref part="R11" gate="G$1" pin="2"/>
 <pinref part="R15" gate="G$1" pin="1"/>
 <pinref part="D11" gate="G$1" pin="C"/>
@@
 <wire x1="185.42" y1="152.4" x2="177.8" y2="152.4" width="0.1524" layer="91"/>
 <wire x1="177.8" y1="152.4" x2="177.8" y2="-45.72" width="0.1524" layer="91"/>
+<pinref part="R11" gate="G$1" pin="1"/>
+<wire x1="185.42" y1="-55.88" x2="185.42" y2="-45.72" width="0.1524" layer="91"/>
 </segment>
 </net>
@@
 <net name="DIG-IN1" class="0">
 <segment>
-<wire x1="215.9" y1="88.9" x2="215.9" y2="86.36" width="0.1524" layer="91"/>
-<wire x1="215.9" y1="86.36" x2="215.9" y2="73.66" width="0.1524" layer="91"/>
-<wire x1="215.9" y1="86.36" x2="223.52" y2="86.36" width="0.1524" layer="91"/>
-<junction x="215.9" y="86.36"/>
-<wire x1="223.52" y1="86.36" x2="223.52" y2="116.84" width="0.1524" layer="91"/>
-<wire x1="223.52" y1="116.84" x2="388.62" y2="116.84" width="0.1524" layer="91"/>
+<wire x1="215.9" y1="73.66" x2="215.9" y2="116.84" width="0.1524" layer="91"/>
+<wire x1="215.9" y1="116.84" x2="388.62" y2="116.84" width="0.1524" layer="91"/>
 <wire x1="388.62" y1="116.84" x2="388.62" y2="76.2" width="0.1524" layer="91"/>
 <junction x="388.62" y="76.2"/>
@@
 <pinref part="Q3" gate="G$1" pin="G"/>
 <wire x1="373.38" y1="76.2" x2="388.62" y2="76.2" width="0.1524" layer="91"/>
-<pinref part="R3" gate="G$1" pin="1"/>
 <wire x1="215.9" y1="73.66" x2="195.58" y2="73.66" width="0.1524" layer="91"/>
 <junction x="215.9" y="73.66"/>
@@
 <wire x1="203.2" y1="152.4" x2="195.58" y2="152.4" width="0.1524" layer="91"/>
 <wire x1="195.58" y1="152.4" x2="195.58" y2="73.66" width="0.1524" layer="91"/>
-</segment>
-</net>
+<pinref part="R3" gate="G$1" pin="2"/>
+<wire x1="215.9" y1="55.88" x2="215.9" y2="73.66" width="0.1524" layer="91"/>
+</segment>
+</net>
