File: Kruispunt/Kruispunt schema v3.brd (EAGLE design)
At the start: 100 x 100.1 mm, 122 parts, among them IC1 74ACT132N, IC2 LM555N, IC3 LM555N, IC4 74AC132N, Q1 BC548, Q10 BC548, Q2 2N3906, Q5 BC548, Q6 2N3906, Q9 BC548, X1 Rood2, X10 Voetgagnersknop1, X11 Voetgangersknop 2 en 1, X12 Groen1, X13 Geel1, X14 Groen2, X4 Rood1, X6 Geel2

Commit message: v3
Parts:
- added R31, R32: 10k, Kruispunt Library:0207/10
- R10, R18: value 1k -> 220
- moved IC4 15.0 mm to (84.5, 42.8)
- moved C10 14.6 mm to (83.9, 57.7)
- moved 17 9.22 mm to (46.4, 43.4)
- moved 13 7.07 mm to (46.6, 36.4)
- moved 11 4.12 mm to (23.6, -2.23)
- moved 10 3.00 mm to (45.5, -3.68)
- moved Q2 3.00 mm to (41.1, 32.7)
- moved JP2 2.83 mm to (52.0, -2.00)
- moved 2 2.24 mm to (30.8, -4.80)
- moved 9 2.24 mm to (94.3, 27.5)
- moved C11 2.24 mm to (83.9, 71.4)
- moved D16 2.00 mm to (84.3, 22.1)
- moved D14 1.41 mm to (77.8, 39.2)
- moved 1 1.00 mm to (61.1, -5.91)
- moved 12 1.00 mm to (47.7, 52.8)
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Connections:
- removed net N$46: ATTINY85.P4, X11.2
- new net N$51: ATTINY85.P4, R31.1, X10.2
- net DIG-IN1: now also R3.2; no longer R3.1
- net DIG-IN2: now also R11.1; no longer R11.2
- net GND: now also R11.2, R3.1, X12.1, X14.1; no longer X12.2, X14.2
- net N$11: now also X12.2; no longer X12.1
- net N$23: now also X14.2; no longer X14.1
- net N$26: now also R32.1, X11.2; no longer X10.2
- net VCC: now also R31.2, R32.2; no longer R11.1, R3.2
Other:
- board text added: "Ard In"
- board text added: "Ard Uit"
- board text added: "Kruispunt V3 Robbe Dierickx 23/04/2019"
- board text added: "Spoel 1"
- board text added: "Spoel 2"
- board text added: "VCC"
- board text removed: "Kruispunt V2 Robbe Dierickx 11/01/19"

Commit message: v3 gerber verslag
Routing:
- net VCC: track 0.00 -> 517.1 mm, vias 0 -> 2
- net N$51: track 0.00 -> 267.9 mm, vias 0 -> 3
- net N$26: track 0.00 -> 184.3 mm, vias 0 -> 2
- net N$47: track 0.00 -> 150.5 mm, vias 0 -> 2
- net N$6: track 0.00 -> 122.9 mm, vias 0 -> 1
- net N$44: track 0.00 -> 122.8 mm, vias 0 -> 2
- net N$48: track 0.00 -> 122.6 mm
- net N$14: track 0.00 -> 122.3 mm, vias 0 -> 4
- net N$11: track 0.00 -> 110.8 mm, vias 0 -> 3
- net DIG-IN1: track 0.00 -> 109.0 mm, vias 0 -> 2
- net N$35: track 0.00 -> 107.4 mm
- net N$20: track 0.00 -> 106.4 mm, vias 0 -> 1
- net N$18: track 0.00 -> 105.5 mm, vias 0 -> 5
- net VCC-LUS: track 0.00 -> 95.6 mm, vias 0 -> 1
- net N$50: track 0.00 -> 92.9 mm, vias 0 -> 1
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