File: Kruispunt/Kruispunt schema v3.sch (EAGLE design)
At the start: 123 parts, among them IC1 74ACT132N, IC2 LM555N, IC3 LM555N, IC4 74AC132N, Q1 BC548, Q10 BC548, Q2 2N3906, Q5 BC548, Q6 2N3906, Q9 BC548, X1 Rood2, X10 Voetgagnersknop1, X11 Voetgangersknop 2 en 1, X12 Groen1, X13 Geel1, X14 Groen2, X4 Rood1, X6 Geel2

Commit message: v3
Parts:
- removed L1, L2: 470µH, Detectielus library:SPOEL
- added R31, R32: 10k, Kruispunt Library:RESISTOR
- added X9: (no value), Kruispunt Library:TERMINAL-5MM-2POLE
- R10, R18: value 1k -> 220
- renumbered PAD1 to 1, PAD10 to 10, PAD11 to 11, PAD12 to 12, PAD13 to 13, PAD14 to 14, PAD15 to 15, PAD16 to 16, PAD17 to 17, PAD18 to 18, PAD19 to 19, PAD2 to 2, PAD3 to 3, PAD4 to 4, PAD5 to 5, PAD6 to 6, PAD7 to 7, PAD8 to 8, PAD9 to 9
Connections:
- removed net N$46: ATTINY85.P4, X11-2.P$2
- new net N$51: ATTINY85.P4, R31.1, X10-2.P$2
- net DIG-IN1: now also R3.2; no longer R3.1
- net DIG-IN2: now also R11.1; no longer R11.2
- net GND: now also R11.2, R3.1, X12-1.P$1, X14-1.P$1, X9-1.P$1; no longer X12-2.P$2, X14-2.P$2
- net LUS-OUT1: no longer L2.1
- net N$11: now also X12-2.P$2; no longer X12-1.P$1
- net N$23: now also X14-2.P$2; no longer X14-1.P$1
- net N$26: now also R32.1, X11-2.P$2; no longer X10-2.P$2
- net N$33: no longer L1.1
- net N48: no longer L2.2
- net N49: no longer L1.2
- net VCC: now also R31.2, R32.2, X9-2.P$2; no longer R11.1, R3.2
Other:
- moved on the sheet: R11, R3, X10-1, X10-2, X11-1, X11-2, X12-1, X12-2, X14-1, X14-2

Commit message: logboek
Other:
- note added: "V3"
- note removed: "V2"
Changed lines of the file:
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@@
 <text x="-16.51" y="41.148" size="2.1844" layer="94">&gt;DRAWING_NAME</text>
 <text x="-16.51" y="35.814" size="2.1844" layer="94">&gt;LAST_DATE_TIME</text>
-<text x="-16.51" y="30.734" size="2.1844" layer="94">V2</text>
+<text x="-16.51" y="30.734" size="2.1844" layer="94">V3</text>
 </plain>
 <instances>
